File: Electronique balance/ruche.kicad_pcb (KiCad board)
At the start: 2 copper layers, 82.8 x 99.9 mm, 155 parts, among them IC1 CN3791, IC2 MAX17048G+, IC3 L86-M33, IC4 SHT41-AD1B-R3, IC5 HX711, IC6 HX711, IC7 HX711, IC8 HX711, J1 Conn_01x02, J10 Conn_01x05, J11 Conn_01x04, J12 Conn_01x04, J13 Micro_SD_Card, J14 Conn_01x03, J15 Conn_01x05, J16 Conn_01x05, J17 Conn_01x04, J18 Conn_01x04, J19 Conn_01x02, J2 Conn_01x05, J3 Conn_01x03, J4 Conn_01x03, J5 Conn_01x04, J6 Conn_01x02, J7 Conn_01x02, J8 Conn_01x03, J9 Conn_01x03, Q1 AO3401A, Q2 MMBT4403, Q3 MMBT4403, Q4 MMBT4403, Q5 MMBT4403, U1 MKRWAN_1310, U2 MS5611-01BA, U3 XC6220B331MR, U4 TCA9548APWR, U5 XC6220B331MR

Commit message: Update
Parts:
- C51: value 10µF -> 0.1µF
- C52: value 0.1µF -> 10µF
Changed lines of the file:
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@@
       (effects (font (size 1 1) (thickness 0.15)))
     )
-    (fp_text value "0.1µF" (at 0 1.68 90) (layer "F.Fab")
+    (fp_text value "10µF" (at 0 1.68 90) (layer "F.Fab")
       (effects (font (size 1 1) (thickness 0.15)))
     )
@@
       (effects (font (size 1 1) (thickness 0.15)))
     )
-    (fp_text value "10µF" (at 0 1.43 90) (layer "F.Fab")
-      (effects (font (size 1 1) (thickness 0.15)))
-    )
+    (fp_text value "0.1µF" (at 0 1.43 90) (layer "F.Fab")
+      (effects (font (size 1 1) (thickness 0.15)))
+    )
