File: Electronique balance/ruche.kicad_sch (KiCad schematic)
At the start: 39 parts, among them IC2 MAX17048G+, IC3 L86-M33, IC4 SHT41-AD1B-R3, J13 Micro_SD_Card, J19 Conn_01x02, U1 MKRWAN_1310, U2 MS5611-01BA, U3 XC6220B331MR, U5 XC6220B331MR

Commit message: Update
Parts:
- renumbered C52 to C51, C51 to C52
Changed lines of the file:
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@@
   (symbol (lib_id "Device:C") (at 40.64 33.02 0) (unit 1)
     (in_bom yes) (on_board yes)
-    (property "Reference" "C51" (id 0) (at 43.561 31.8516 0)
+    (property "Reference" "C52" (id 0) (at 43.561 31.8516 0)
       (effects (font (size 1.27 1.27)) (justify left))
     )
@@
   (symbol (lib_id "Device:C") (at 50.8 33.02 0) (unit 1)
     (in_bom yes) (on_board yes)
-    (property "Reference" "C52" (id 0) (at 53.721 31.8516 0)
+    (property "Reference" "C51" (id 0) (at 53.721 31.8516 0)
       (effects (font (size 1.27 1.27)) (justify left))
     )
@@
       (reference "C50") (unit 1) (value "0.1µF") (footprint "Capacitor_SMD:C_0603_1608Metric")
     )
+    (path "/fd8286f5-83f2-4c75-b09d-fdd0c502a928"
+      (reference "C51") (unit 1) (value "0.1µF") (footprint "Capacitor_SMD:C_0805_2012Metric")
+    )
     (path "/4bd821f2-0707-4078-b490-ee80c8fe83b7"
-      (reference "C51") (unit 1) (value "10µF") (footprint "Capacitor_SMD:C_0603_1608Metric")
-    )
-    (path "/fd8286f5-83f2-4c75-b09d-fdd0c502a928"
-      (reference "C52") (unit 1) (value "0.1µF") (footprint "Capacitor_SMD:C_0805_2012Metric")
+      (reference "C52") (unit 1) (value "10µF") (footprint "Capacitor_SMD:C_0603_1608Metric")
     )
     (path "/d2746501-2960-4618-ba16-fa886c4044e2"
