File: Electronique balance/rucheb.kicad_sch (KiCad schematic)
At the start: 23 parts, among them IC1 CN3791, J1 Conn_01x02, Q1 AO3401A

Commit message: Update
Parts:
- R1: value 2K -> 10K
Changed lines of the file:
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@@
       (effects (font (size 1.27 1.27)) (justify left))
     )
-    (property "Value" "2K" (id 1) (at 43.688 77.343 0)
+    (property "Value" "10K" (id 1) (at 43.688 77.343 0)
       (effects (font (size 1.27 1.27)) (justify left))
     )
